File: MacroPad.kicad_sch (KiCad schematic)
At the start: 45 parts, among them J2 AVR-ISP-6, SW1 SW_Push, U1 ATmega32U4-A, Y1 16MHz

Commit message: production files
Parts:
- C1, C2: LCSC (none) -> C1804
- C3: LCSC (none) -> C116352
- C4, C5, C6, C7: LCSC (none) -> C1711
- C8: LCSC (none) -> C307520
- D1, D10, D11, D12, D3, D4, D5, D6, D7, D8, D9: LCSC (none) -> C77978
- D13: LCSC (none) -> C2827688
- F1: LCSC (none) -> C5118830
- MX1, MX10, MX11, MX12, MX2, MX3, MX4, MX5, MX6, MX7, MX8, MX9: LCSC (none) -> C5156480
- R1, R5: LCSC (none) -> C100047
- R2, R6: LCSC (none) -> C105874
- R3, R4: LCSC (none) -> C114231
- SW1: LCSC (none) -> C2689521
- U1: LCSC (none) -> C44854
- USB1: LCSC (none) -> C165948
- Y1: LCSC (none) -> C2650477
Changed lines of the file:
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@@
+      (effects (font (size 1.27 1.27)) hide)
+    )
+    (property "LCSC" "C100047" (at 83.82 86.36 90)
       (effects (font (size 1.27 1.27)) hide)
     )
@@
       (effects (font (size 1.27 1.27)) hide)
     )
+    (property "LCSC" "C1804" (at 23.495 38.1 90)
+      (effects (font (size 1.27 1.27)) hide)
+    )
     (pin "1")
     (pin "2")
@@
     )
     (property "Datasheet" "~" (at 36.195 40.64 0)
+      (effects (font (size 1.27 1.27)) hide)
+    )
+    (property "LCSC" "C2650477" (at 36.195 40.64 90)
       (effects (font (size 1.27 1.27)) hide)
     )
@@
       (effects (font (size 1.524 1.524)) hide)
     )
+    (property "LCSC" "C5156480" (at 264.795 66.04 0)
+      (effects (font (size 1.27 1.27)) hide)
+    )
     (pin "1")
     (pin "2")
@@
       (effects (font (size 1.27 1.27)) hide)
     )
+    (property "LCSC" "C1804" (at 23.495 43.18 90)
+      (effects (font (size 1.27 1.27)) hide)
+    )
     (pin "1")
     (pin "2")
@@
     )
     (property "Datasheet" "~" (at 26.035 58.42 0)
+      (effects (font (size 1.27 1.27)) hide)
+    )
+    (property "LCSC" "C114231" (at 26.035 58.42 90)
       (effects (font (size 1.27 1.27)) hide)
     )
@@
       (effects (font (size 1.524 1.524)) hide)
     )
+    (property "LCSC" "C5156480" (at 264.795 44.45 0)
+      (effects (font (size 1.27 1.27)) hide)
+    )
     (pin "1")
     (pin "2")
@@
       (effects (font (size 1.27 1.27)) hide)
     )
+    (property "LCSC" "C77978" (at 263.525 74.295 90)
+      (effects (font (size 1.27 1.27)) hide)
+    )
     (pin "1")
     (pin "2")
@@
     )
     (property "Sim.Pins" "1=K 2=A" (at 263.525 118.745 0)
+      (effects (font (size 1.27 1.27)) hide)
+    )
+    (property "LCSC" "C77978" (at 263.525 118.745 90)
       (effects (font (size 1.27 1.27)) hide)
     )
@@
       (effects (font (size 1.524 1.524)) hide)
     )
+    (property "LCSC" "C5156480" (at 236.855 66.04 0)
+      (effects (font (size 1.27 1.27)) hide)
+    )
     (pin "1")
     (pin "2")
@@
     )
     (property "Sim.Pins" "1=K 2=A" (at 235.585 95.885 0)
+      (effects (font (size 1.27 1.27)) hide)
+    )
+    (property "LCSC" "C77978" (at 235.585 95.885 90)
       (effects (font (size 1.27 1.27)) hide)
     )
@@
       (effects (font (size 1.27 1.27)) hide)
     )
+    (property "LCSC" "C5118830" (at 144.145 45.72 90)
+      (effects (font (size 1.27 1.27)) hide)
+    )
     (pin "1")
     (pin "2")
@@
       (effects (font (size 1.27 1.27)) hide)
     )
+    (property "LCSC" "C116352" (at 39.37 68.58 0)
+      (effects (font (size 1.27 1.27)) hide)
+    )
     (pin "1")
     (pin "2")
@@
       (effects (font (size 1.27 1.27)) hide)
     )
+    (property "LCSC" "C105874" (at 152.4 50.8 90)
+      (effects (font (size 1.27 1.27)) hide)
+    )
     (pin "1")
     (pin "2")
@@
     )
     (property "Datasheet" "~" (at 31.75 27.94 0)
+      (effects (font (size 1.27 1.27)) hide)
+    )
+    (property "LCSC" "C2689521" (at 31.75 33.02 0)
       (effects (font (size 1.27 1.27)) hide)
     )
@@
     )
     (property "Datasheet" "http://ww1.microchip.com/downloads/en/DeviceDoc/Atmel-7766-8-bit-AVR-ATmega16U4-32U4_Datasheet.pdf" (at 59.055 71.12 0)
+      (effects (font (size 1.27 1.27)) hide)
+    )
+    (property "LCSC" "C44854" (at 59.055 71.12 0)
       (effects (font (size 1.27 1.27)) hide)
     )
@@
       (effects (font (size 1.524 1.524)) hide)
     )
+    (property "LCSC" "C5156480" (at 250.825 66.04 0)
+      (effects (font (size 1.27 1.27)) hide)
+    )
     (pin "1")
     (pin "2")
@@
     )
     (property "Sim.Pins" "1=K 2=A" (at 263.525 52.705 0)
+      (effects (font (size 1.27 1.27)) hide)
+    )
+    (property "LCSC" "C77978" (at 263.525 52.705 90)
       (effects (font (size 1.27 1.27)) hide)
     )
@@
       (effects (font (size 1.524 1.524)) hide)
     )
+    (property "LCSC" "C5156480" (at 236.855 110.49 0)
+      (effects (font (size 1.27 1.27)) hide)
+    )
     (pin "1")
     (pin "2")
@@
       (effects (font (size 1.27 1.27)) hide)
     )
+    (property "LCSC" "C77978" (at 249.555 95.885 90)
+      (effects (font (size 1.27 1.27)) hide)
+    )
     (pin "1")
     (pin "2")
@@
     )
     (property "Datasheet" "https://assets.nexperia.com/documents/data-sheet/PRTR5V0U2X.pdf" (at 127.889 82.55 0)
+      (effects (font (size 1.27 1.27)) hide)
+    )
+    (property "LCSC" "C2827688" (at 126.365 82.55 0)
       (effects (font (size 1.27 1.27)) hide)
     )
@@
       (effects (font (size 1.27 1.27)) hide)
     )
+    (property "LCSC" "C77978" (at 235.585 118.745 90)
+      (effects (font (size 1.27 1.27)) hide)
+    )
     (pin "1")
     (pin "2")
@@
       (effects (font (size 1.27 1.27)) hide)
     )
+    (property "LCSC" "C77978" (at 249.555 74.295 90)
+      (effects (font (size 1.27 1.27)) hide)
+    )
     (pin "1")
     (pin "2")
@@
     )
     (property "Sim.Pins" "1=K 2=A" (at 249.555 52.705 0)
+      (effects (font (size 1.27 1.27)) hide)
+    )
+    (property "LCSC" "C77978" (at 249.555 52.705 90)
       (effects (font (size 1.27 1.27)) hide)
     )
@@
       (effects (font (size 1.524 1.524)) hide)
     )
+    (property "LCSC" "C5156480" (at 250.825 87.63 0)
+      (effects (font (size 1.27 1.27)) hide)
+    )
     (pin "1")
     (pin "2")
@@
     )
     (property "Sim.Pins" "1=K 2=A" (at 249.555 118.745 0)
+      (effects (font (size 1.27 1.27)) hide)
+    )
+    (property "LCSC" "C77978" (at 249.555 118.745 90)
       (effects (font (size 1.27 1.27)) hide)
     )
@@
     (property "Datasheet" "" (at 165.1 57.15 0)
       (effects (font (size 1.524 1.524)) hide)
+    )
+    (property "LCSC" "C165948" (at 165.1 57.15 0)
+      (effects (font (size 1.27 1.27)) hide)
     )
     (pin "1")
@@
       (effects (font (size 1.27 1.27)) hide)
     )
+    (property "LCSC" "C105874" (at 152.4 66.04 90)
+      (effects (font (size 1.27 1.27)) hide)
+    )
     (pin "1")
     (pin "2")
@@
       (effects (font (size 1.27 1.27)) hide)
     )
+    (property "LCSC" "C1711" (at 97.155 17.78 0)
+      (effects (font (size 1.27 1.27)) hide)
+    )
     (pin "1")
     (pin "2")
@@
       (effects (font (size 1.524 1.524)) hide)
     )
+    (property "LCSC" "C5156480" (at 236.855 87.63 0)
+      (effects (font (size 1.27 1.27)) hide)
+    )
     (pin "1")
     (pin "2")
@@
     )
     (property "Datasheet" "~" (at 26.035 60.96 0)
+      (effects (font (size 1.27 1.27)) hide)
+    )
+    (property "LCSC" "C114231" (at 26.035 60.96 90)
       (effects (font (size 1.27 1.27)) hide)
     )
@@
       (effects (font (size 1.524 1.524)) hide)
     )
+    (property "LCSC" "C5156480" (at 264.795 87.63 0)
+      (effects (font (size 1.27 1.27)) hide)
+    )
     (pin "1")
     (pin "2")
@@
       (effects (font (size 1.524 1.524)) hide)
     )
+    (property "LCSC" "C5156480" (at 250.825 110.49 0)
+      (effects (font (size 1.27 1.27)) hide)
+    )
     (pin "1")
     (pin "2")
@@
       (effects (font (size 1.524 1.524)) hide)
     )
+    (property "LCSC" "C5156480" (at 264.795 110.49 0)
+      (effects (font (size 1.27 1.27)) hide)
+    )
     (pin "1")
     (pin "2")
@@
     )
     (property "Datasheet" "~" (at 38.1 24.765 0)
+      (effects (font (size 1.27 1.27)) hide)
+    )
+    (property "LCSC" "C100047" (at 38.1 24.765 0)
       (effects (font (size 1.27 1.27)) hide)
     )
@@
       (effects (font (size 1.27 1.27)) hide)
     )
+    (property "LCSC" "C307520" (at 106.045 17.78 0)
+      (effects (font (size 1.27 1.27)) hide)
+    )
     (pin "1")
     (pin "2")
@@
       (effects (font (size 1.524 1.524)) hide)
     )
+    (property "LCSC" "C5156480" (at 236.855 44.45 0)
+      (effects (font (size 1.27 1.27)) hide)
+    )
     (pin "1")
     (pin "2")
@@
       (effects (font (size 1.524 1.524)) hide)
     )
+    (property "LCSC" "C5156480" (at 250.825 44.45 0)
+      (effects (font (size 1.27 1.27)) hide)
+    )
     (pin "1")
     (pin "2")
@@
       (effects (font (size 1.27 1.27)) hide)
     )
+    (property "LCSC" "C1711" (at 79.375 17.78 0)
+      (effects (font (size 1.27 1.27)) hide)
+    )
     (pin "1")
     (pin "2")
@@
       (effects (font (size 1.27 1.27)) hide)
     )
+    (property "LCSC" "C77978" (at 263.525 95.885 90)
+      (effects (font (size 1.27 1.27)) hide)
+    )
     (pin "1")
     (pin "2")
@@
     )
     (property "Sim.Pins" "1=K 2=A" (at 235.585 52.705 0)
+      (effects (font (size 1.27 1.27)) hide)
+    )
+    (property "LCSC" "C77978" (at 235.585 52.705 90)
       (effects (font (size 1.27 1.27)) hide)
     )
@@
       (effects (font (size 1.27 1.27)) hide)
     )
+    (property "LCSC" "C1711" (at 70.485 17.78 0)
+      (effects (font (size 1.27 1.27)) hide)
+    )
     (pin "1")
     (pin "2")
@@
       (effects (font (size 1.27 1.27)) hide)
     )
+    (property "LCSC" "C1711" (at 88.265 17.78 0)
+      (effects (font (size 1.27 1.27)) hide)
+    )
